Commit message: changed how to set static

File: husky_description/urdf/husky_velodyne.urdf.xacro (robot description, xacro)
@@ -33,11 +33,10 @@
 -->
 <robot name="husky" xmlns:xacro="http://ros.org/wiki/xacro">
-    <xacro:arg name="static" default="true" />
-    <xacro:property name="static" value="$(arg static)" />
-    <xacro:macro name="static_macro">
-        <gazebo>
-            <static>1</static>
-        </gazebo>
-    </xacro:macro>
+    <xacro:arg name="static" default="$(optenv HUSKY_STATIC 1)" />
+    <xacro:if value="$(arg static)">
+    <gazebo>
+      <static>1</static>
+    </gazebo>
+    </xacro:if>
     <xacro:arg name="laser_enabled" default="false" />
     <xacro:arg name="laser_xyz" default="$(optenv HUSKY_LMS1XX_XYZ 0.2206 0.0 0.00635)" />
@@ -223,9 +222,6 @@
     <xacro:include filename="$(find velodyne_description)/urdf/VLP-16.urdf.xacro" />
     <xacro:VLP-16 parent="base_link" name="velodyne" topic="/velodyne_points" organize_cloud="false"
-        hz="10" samples="720" gpu="false">
+        hz="10" gpu="true">
         <origin xyz="0 0 0.4" rpy="0 0 0" />
     </xacro:VLP-16>
-    <xacro:if value="${static}">
-        <xacro:static_macro />
-    </xacro:if>
 </robot>
